Commit message: Swap vision camera from D435 to L515 LiDAR
- Body: box (90×25×25 mm) → cylinder (61 mm ⌀ × 26 mm)
- H FOV: 60° → 70° (1.2217 rad)
- Clip near: 0.1 m → 0.25 m  (L515 minimum range)
- Clip far: 3.0 m → 9.0 m
- Depth noise: σ=0.002 m → σ=0.003 m (ToF is uniform; stereo has edge falloff)
- Sensor name: d435_vision → l515_vision
- Resolution kept at 640×480 for WSL2 performance (FOV identical to 1024×768)

https://claude.ai/code/session_014jKiKFNFx2wbEBY1JDbtYJ

File: arctos_gazebo/urdf/vision_camera.urdf.xacro (robot description, xacro)
@@ -2,11 +2,19 @@
 <!--
   vision_camera.urdf.xacro
-  Standalone Intel RealSense D435 camera for the vision-only simulation.
-  No arm, no controllers — just a static camera fixed to the world looking
-  at a tabletop workspace.
+  Standalone Intel RealSense L515 LiDAR camera for the vision-only simulation.
+  The L515 uses a LiDAR Time-of-Flight sensor rather than the D435's stereo
+  infrared.  Key simulation differences vs D435:
+    - Cylindrical body (61 mm ⌀ × 26 mm) instead of a bar
+    - 70° × 55° FOV (narrower than D435's 86° × 57°)
+    - Minimum range 0.25 m  ← objects closer than this have no depth return
+    - Depth noise σ = 0.003 m (~3 mm) vs D435's ~10–20 mm
+    - Native depth resolution 1024 × 768; downscaled to 640 × 480 here for
+      WSL2 rendering performance (FOV is preserved exactly)
   Camera mount:
     xyz = "0.4 0.0 0.42"   — 40 cm in front of table centre, 42 cm up
     rpy = "0 0.7 3.14159"  — pitched ~40° downward, facing -X (toward table)
-  Adjust the camera_joint origin to reposition the camera view.
+    At this distance the table (0.6 m wide) fits comfortably in the 70° FOV.
+    Nearest table point is ~0.35 m — just above the 0.25 m minimum range.
+  Adjust the camera_world_joint origin to reposition the camera view.
   Topics bridged by ros_gz_bridge (via vision_sim.launch.py):
     /vision/image          — 640×480 RGB
@@ -18,10 +26,10 @@
   <!-- World anchor — fixed to the SDF world frame by Gazebo -->
   <link name="world"/>
-  <!-- Camera body: approximate D435 dimensions (90×25×25 mm) -->
+  <!-- Camera body: L515 form factor — 61 mm diameter × 26 mm tall cylinder -->
   <link name="camera_link">
     <visual>
       <origin xyz="0 0 0" rpy="0 0 0"/>
       <geometry>
-        <box size="0.025 0.090 0.025"/>
+        <cylinder radius="0.0305" length="0.026"/>
       </geometry>
       <material name="realsense_body">
@@ -30,6 +38,6 @@
     </visual>
     <inertial>
-      <mass value="0.072"/>
-      <inertia ixx="0.000038" iyy="0.000005" izz="0.000038"
+      <mass value="0.100"/>  <!-- L515: 100 g -->
+      <inertia ixx="0.000041" iyy="0.000041" izz="0.000047"
                ixy="0" ixz="0" iyz="0"/>
     </inertial>
@@ -54,28 +62,36 @@
   </joint>
   <!--
-    Intel RealSense D435 RGBD sensor — 640×480, 60° horizontal FOV.
-    Narrower than the 848-wide mode so the full table fits in frame
-    at this mount distance.
-    Depth noise: Gaussian σ=0.002 m (~2 mm at 0.5 m range).
+    Intel RealSense L515 LiDAR sensor.
+    Spec        Real L515        Simulated here
+    ---------   --------         ----------------
+    H FOV       70°              70° (1.2217 rad)
+    V FOV       55°              55° (aspect ratio 640×480 ≈ 4:3 ≈ 56°)
+    Depth res   1024 × 768       640 × 480  (same FOV, lighter for WSL2)
+    Min range   0.25 m           0.25 m  ← objects closer give no return
+    Max range   9 m              9 m
+    Noise       ~3–5 mm          σ = 0.003 m (Gaussian)
+    Rate        30 fps           30 fps
+    The ToF nature means noise is uniform across the image (no stereo
+    falloff toward edges), so a single Gaussian model is appropriate.
     All topics are published under the "vision" prefix so they don't
     collide with the arm simulation's "/camera/*" topics.
   -->
   <gazebo reference="camera_optical_frame">
-    <sensor name="d435_vision" type="rgbd_camera">
+    <sensor name="l515_vision" type="rgbd_camera">
       <camera>
-        <horizontal_fov>1.0472</horizontal_fov>  <!-- 60° -->
+        <horizontal_fov>1.2217</horizontal_fov>  <!-- 70° -->
         <image>
           <width>640</width>
-          <height>480</height>
+          <height>480</height>   <!-- 4:3 → V FOV ≈ 55°; matches real L515 -->
           <format>R8G8B8</format>
         </image>
         <clip>
-          <near>0.1</near>
-          <far>3.0</far>
+          <near>0.25</near>   <!-- L515 minimum range: 0.25 m -->
+          <far>9.0</far>
         </clip>
         <noise>
           <type>gaussian</type>
           <mean>0.0</mean>
-          <stddev>0.002</stddev>
+          <stddev>0.003</stddev>  <!-- ~3 mm; ToF is far more precise than stereo -->
         </noise>
       </camera>
