Commit message: Fix Gazebo mesh resolution and RViz RobotModel error
- Set GZ_SIM_RESOURCE_PATH from AMENT_PREFIX_PATH in sim.launch.py so
  Gazebo Harmonic can resolve package:// mesh URIs (base_link.stl etc.)
- Make RViz config optional: fall back gracefully if arctos.rviz absent
- Replace undefined material 'Black' with inline RGBA color in
  arctos_sim.xacro to fix URDF parse warnings

https://claude.ai/code/session_014jKiKFNFx2wbEBY1JDbtYJ

File: arctos_gazebo/urdf/arctos_sim.xacro (robot description, xacro)
@@ -149,5 +149,5 @@
         <box size="0.05 0.05 0.9"/>
       </geometry>
-      <material name="Black"/>
+      <material name="black"><color rgba="0.1 0.1 0.1 1.0"/></material>
     </visual>
     <collision>
@@ -175,5 +175,5 @@
         <box size="0.1 0.04 0.04"/>
       </geometry>
-      <material name="Black"/>
+      <material name="black"><color rgba="0.1 0.1 0.1 1.0"/></material>
     </visual>
     <inertial>

Commit message: fix(arctos_sim.xacro): remove dual world-child and spurious <ros> block
Two bugs that together caused the Gazebo model spawn to abort:

1. DUAL-WORLD-CHILD: arctos.xacro already attaches base_link to the
   'world' link via world_joint.  Adding a second fixed joint from 'world'
   to camera_stand created two kinematic chains rooted at 'world'.
   Gazebo Harmonic's URDF→SDF converter does not support multiple children
   of the world link in a single model, so the entire spawn was silently
   aborted and the robot never appeared in Gazebo.

   Fix: remove the camera stand from the robot URDF entirely.  Camera
   placement will be handled as a child of the robot end-effector link
   (eye-in-hand configuration), keeping a single kinematic chain.

2. SPURIOUS <ros> BLOCK: the <ros><remapping>...</remapping></ros> section
   inside the gz_ros2_control plugin element is not a recognised tag in
   gz_ros2_control for Harmonic and can cause the plugin to fail to
   initialise, preventing controller_manager from starting.  Removed.

https://claude.ai/code/session_014jKiKFNFx2wbEBY1JDbtYJ

File: arctos_gazebo/urdf/arctos_sim.xacro (robot description, xacro)
@@ -127,116 +127,5 @@
             name="gz_ros2_control::GazeboSimROS2ControlPlugin">
       <parameters>$(find arctos_gazebo)/config/sim_controllers.yaml</parameters>
-      <ros>
-        <remapping>~/robot_description:=/robot_description</remapping>
-      </ros>
     </plugin>
   </gazebo>
-  <!-- ================================================================== -->
-  <!-- Depth camera on a fixed stand                                       -->
-  <!--                                                                     -->
-  <!-- Placement: 0.8 m in front of the robot base, 0.9 m high, angled   -->
-  <!-- ~37° downward so the lens covers the full workspace.               -->
-  <!--                                                                     -->
-  <!-- Coordinate note: Gazebo rgbd_camera looks along the link's +X axis. -->
-  <!-- The camera_joint rpy rotates the stand top so +X faces the robot.  -->
-  <!-- Fine-tune the pitch (second rpy value) to adjust the field of view. -->
-  <!-- ================================================================== -->
-  <!-- Vertical stand pole -->
-  <link name="camera_stand">
-    <visual>
-      <origin xyz="0 0 0.45" rpy="0 0 0"/>
-      <geometry>
-        <box size="0.05 0.05 0.9"/>
-      </geometry>
-      <material name="black"><color rgba="0.1 0.1 0.1 1.0"/></material>
-    </visual>
-    <collision>
-      <origin xyz="0 0 0.45" rpy="0 0 0"/>
-      <geometry>
-        <box size="0.05 0.05 0.9"/>
-      </geometry>
-    </collision>
-    <inertial>
-      <mass value="1.0"/>
-      <inertia ixx="0.068" iyy="0.068" izz="0.0001" ixy="0" ixz="0" iyz="0"/>
-    </inertial>
-  </link>
-  <!-- Stand is fixed to world at (0.8, 0, 0) -->
-  <joint name="camera_stand_joint" type="fixed">
-    <parent link="world"/>
-    <child link="camera_stand"/>
-    <origin xyz="0.8 0.0 0.0" rpy="0 0 0"/>
-  </joint>
-  <!-- Camera housing at the top of the stand -->
-  <link name="camera_link">
-    <visual>
-      <origin xyz="0 0 0" rpy="0 0 0"/>
-      <geometry>
-        <box size="0.1 0.04 0.04"/>
-      </geometry>
-      <material name="black"><color rgba="0.1 0.1 0.1 1.0"/></material>
-    </visual>
-    <inertial>
-      <mass value="0.1"/>
-      <inertia ixx="0.00001" iyy="0.00001" izz="0.00001" ixy="0" ixz="0" iyz="0"/>
-    </inertial>
-  </link>
-  <!--
-    Rotate the camera to face the robot.
-    rpy="0 0.6435 3.14159":
-      - 3.14159 (yaw 180°) : turns the camera to face -X (toward the robot)
-      - 0.6435  (pitch +37°): tilts the lens downward toward the workspace
-    Adjust these values if you want a different viewing angle.
-  -->
-  <joint name="camera_joint" type="fixed">
-    <parent link="camera_stand"/>
-    <child link="camera_link"/>
-    <origin xyz="0 0 0.9" rpy="0 0.6435 3.14159"/>
-  </joint>
-  <!--
-    Optical frame: ROS camera convention has Z forward, X right, Y down.
-    This extra fixed joint converts from the standard ROS body frame
-    (X forward, Y left, Z up) used by camera_link.
-  -->
-  <link name="camera_optical_frame"/>
-  <joint name="camera_optical_joint" type="fixed">
-    <parent link="camera_link"/>
-    <child link="camera_optical_frame"/>
-    <origin xyz="0 0 0" rpy="-1.5708 0 -1.5708"/>
-  </joint>
-  <!-- ================================================================== -->
-  <!-- rgbd_camera sensor attached to camera_optical_frame                 -->
-  <!-- Publishes to Gazebo topics:                                         -->
-  <!--   /camera/image         (RGB)                                       -->
-  <!--   /camera/depth_image   (depth, float32)                            -->
-  <!--   /camera/camera_info                                               -->
-  <!--   /camera/points        (PointCloud2)                               -->
-  <!-- The ros_gz_bridge in sim.launch.py forwards these into ROS2.        -->
-  <!-- ================================================================== -->
-  <gazebo reference="camera_optical_frame">
-    <sensor name="depth_camera" type="rgbd_camera">
-      <camera>
-        <horizontal_fov>1.047</horizontal_fov>  <!-- 60 degrees -->
-        <image>
-          <width>640</width>
-          <height>480</height>
-          <format>R8G8B8</format>
-        </image>
-        <clip>
-          <near>0.1</near>
-          <far>5.0</far>
-        </clip>
-        <noise>
-          <type>gaussian</type>
-          <mean>0.0</mean>
-          <stddev>0.007</stddev>
-        </noise>
-      </camera>
-      <always_on>true</always_on>
-      <update_rate>30</update_rate>
-      <visualize>true</visualize>
-      <topic>camera</topic>
-      <gz_frame_id>camera_optical_frame</gz_frame_id>
-    </sensor>
-  </gazebo>
 </robot>

Commit message: feat(arctos_sim.xacro): add eye-in-hand RGBD camera on Gripper_1
Mounts an rgbd_camera sensor as part of the robot kinematic chain:

  Gripper_1 → (camera_joint, fixed) → camera_link
  camera_link → (camera_optical_joint, fixed) → camera_optical_frame

This avoids the dual-world-child problem that caused the previous
camera_stand approach to abort the Gazebo model spawn.  The camera is
now part of the single world→base_link→…→Gripper_1→camera chain,
which converts cleanly to SDF.

Default mount: 6 cm forward + 4 cm above Gripper_1 origin, pitched 30°
downward toward the grasp point.  Adjust camera_joint origin xyz/rpy
to match the physical camera position on the real robot.

Near clip: 0.05 m (close-range grasping)
Far  clip: 1.5  m (covers full Arctos workspace)

Gazebo topics (bridged by ros_gz_bridge):
  /camera/image, /camera/depth_image, /camera/camera_info, /camera/points

https://claude.ai/code/session_014jKiKFNFx2wbEBY1JDbtYJ

File: arctos_gazebo/urdf/arctos_sim.xacro (robot description, xacro)
@@ -129,3 +129,76 @@
     </plugin>
   </gazebo>
+  <!-- ================================================================== -->
+  <!-- Eye-in-hand RGBD camera mounted on the robot end effector           -->
+  <!--                                                                     -->
+  <!-- Parent link: Gripper_1 (child of C_joint, parent of jaw joints).   -->
+  <!--                                                                     -->
+  <!-- camera_link      — physical camera body; Gazebo camera looks along  -->
+  <!--                    its +X axis, so rpy below aims the sensor.       -->
+  <!-- camera_optical_frame — ROS camera convention (Z fwd, X right, Y↓)  -->
+  <!--                                                                     -->
+  <!-- ADJUST origin xyz/rpy on camera_joint to match your actual camera   -->
+  <!-- mount position.  Current default:                                   -->
+  <!--   xyz="0.06 0 0.04"  — 6 cm forward, 4 cm above gripper origin    -->
+  <!--   rpy="0 0.5236 0"   — pitched 30° downward to see grasp point     -->
+  <!-- ================================================================== -->
+  <!-- Camera body (small box, visible in RViz/Gazebo) -->
+  <link name="camera_link">
+    <visual>
+      <origin xyz="0 0 0" rpy="0 0 0"/>
+      <geometry>
+        <box size="0.04 0.04 0.02"/>
+      </geometry>
+      <material name="camera_dark">
+        <color rgba="0.2 0.2 0.2 1.0"/>
+      </material>
+    </visual>
+    <inertial>
+      <mass value="0.05"/>
+      <inertia ixx="0.000001" iyy="0.000001" izz="0.000001"
+               ixy="0" ixz="0" iyz="0"/>
+    </inertial>
+  </link>
+  <joint name="camera_joint" type="fixed">
+    <parent link="Gripper_1"/>
+    <child link="camera_link"/>
+    <!-- 6 cm forward along gripper X, 4 cm above, pitched 30° down toward grasp -->
+    <origin xyz="0.06 0.0 0.04" rpy="0 0.5236 0"/>
+  </joint>
+  <!-- ROS optical frame: Z forward, X right, Y down -->
+  <link name="camera_optical_frame"/>
+  <joint name="camera_optical_joint" type="fixed">
+    <parent link="camera_link"/>
+    <child link="camera_optical_frame"/>
+    <origin xyz="0 0 0" rpy="-1.5708 0 -1.5708"/>
+  </joint>
+  <!-- RGBD sensor (Gazebo Harmonic).                                      -->
+  <!-- Near clip 0.05 m suits close-range grasping; far 1.5 m covers the  -->
+  <!-- full reachable workspace of the Arctos arm.                         -->
+  <gazebo reference="camera_optical_frame">
+    <sensor name="depth_camera" type="rgbd_camera">
+      <camera>
+        <horizontal_fov>1.047</horizontal_fov>  <!-- 60° FOV -->
+        <image>
+          <width>640</width>
+          <height>480</height>
+          <format>R8G8B8</format>
+        </image>
+        <clip>
+          <near>0.05</near>
+          <far>1.5</far>
+        </clip>
+        <noise>
+          <type>gaussian</type>
+          <mean>0.0</mean>
+          <stddev>0.007</stddev>
+        </noise>
+      </camera>
+      <always_on>true</always_on>
+      <update_rate>30</update_rate>
+      <visualize>true</visualize>
+      <topic>camera</topic>
+      <gz_frame_id>camera_optical_frame</gz_frame_id>
+    </sensor>
+  </gazebo>
 </robot>

Commit message: feat(camera): replace eye-in-hand with base-fixed Intel RealSense D435
- Move camera parent from Gripper_1 to base_link so the sensor has a
  stable world-fixed viewpoint of the entire arm workspace
- Update sensor to match D435 848×480 depth mode specs:
    horizontal FOV 86° (1.5009 rad), near 0.105 m, far 10.0 m,
    Gaussian depth noise σ = 0.003 m, 30 Hz, visual body 90×25×25 mm
- Enable gz-sim-sensors-system (ogre2) in arctos_world.sdf now that
  robot spawning is confirmed working; env vars in launch file handle
  WSL2 software-rendering compatibility
- Add depth_image_proc/point_cloud_xyzrgb node to sim.launch.py to
  generate an organised XYZRGB PointCloud2 at /camera/points_registered,
  which preserves 2-D pixel topology needed by PCL surface segmentation
- Add depth_image_proc exec_depend to package.xml

https://claude.ai/code/session_014jKiKFNFx2wbEBY1JDbtYJ

File: arctos_gazebo/urdf/arctos_sim.xacro (robot description, xacro)
@@ -7,5 +7,6 @@
        CAN-based ArctosInterface used on real hardware)
     2. Gazebo gz_ros2_control system plugin
-    3. Eye-in-hand RGBD camera fixed to Gripper_1 (end effector)
+    3. Intel RealSense D435 RGBD camera fixed to base_link (world-fixed
+       viewpoint covering the full arm workspace)
 -->
 <robot xmlns:xacro="http://www.ros.org/wiki/xacro" name="arctos_sim">
@@ -130,41 +131,56 @@
   </gazebo>
   <!-- ================================================================== -->
-  <!-- Eye-in-hand RGBD camera mounted on the robot end effector           -->
-  <!--                                                                     -->
-  <!-- Parent link: Gripper_1 (child of C_joint, parent of jaw joints).   -->
-  <!--                                                                     -->
-  <!-- camera_link      — physical camera body; Gazebo camera looks along  -->
-  <!--                    its +X axis, so rpy below aims the sensor.       -->
-  <!-- camera_optical_frame — ROS camera convention (Z fwd, X right, Y↓)  -->
-  <!--                                                                     -->
-  <!-- ADJUST origin xyz/rpy on camera_joint to match your actual camera   -->
-  <!-- mount position.  Current default:                                   -->
-  <!--   xyz="0.06 0 0.04"  — 6 cm forward, 4 cm above gripper origin    -->
-  <!--   rpy="0 0.5236 0"   — pitched 30° downward to see grasp point     -->
-  <!-- ================================================================== -->
-  <!-- Camera body (small box, visible in RViz/Gazebo) -->
+  <!-- Intel RealSense D435 — base-fixed, looking at the arm workspace    -->
+  <!--                                                                     -->
+  <!-- Parent link: base_link (fixed relative to the world — the arm's    -->
+  <!-- base does not move, so this camera has a stable viewpoint of the   -->
+  <!-- entire workspace regardless of arm pose).                           -->
+  <!--                                                                     -->
+  <!-- Mount position (adjust to suit your physical setup):               -->
+  <!--   xyz="-0.08 0.0 0.18"  — 8 cm behind, 18 cm above base origin    -->
+  <!--   rpy="0 0.35 0"        — pitched ~20° forward to centre the FOV  -->
+  <!--                            on the arm's reachable workspace         -->
+  <!--                                                                     -->
+  <!-- D435 depth sensor parameters (848×480 mode):                       -->
+  <!--   Horizontal FOV : 86°  (1.5009 rad)                               -->
+  <!--   Vertical FOV   : 57°  (0.9948 rad, implied by 848×480 aspect)   -->
+  <!--   Min depth      : 0.105 m                                          -->
+  <!--   Max depth      : 10.0 m                                           -->
+  <!--   Frame rate     : 30 Hz                                            -->
+  <!--   Depth noise    : Gaussian σ = 0.003 m (≈ D435 at ~1 m)          -->
+  <!--                                                                     -->
+  <!-- Topics (via ros_gz_bridge):                                         -->
+  <!--   /camera/image        — 848×480 RGB                               -->
+  <!--   /camera/depth_image  — 848×480 float32 depth (metres)            -->
+  <!--   /camera/camera_info  — intrinsics                                 -->
+  <!--   /camera/points       — XYZRGB PointCloud2                        -->
+  <!-- ================================================================== -->
+  <!-- Camera body: D435 is 90×25×25 mm; approximate as a flat box -->
   <link name="camera_link">
     <visual>
       <origin xyz="0 0 0" rpy="0 0 0"/>
       <geometry>
-        <box size="0.04 0.04 0.02"/>
+        <box size="0.025 0.090 0.025"/>
       </geometry>
-      <material name="camera_dark">
-        <color rgba="0.2 0.2 0.2 1.0"/>
+      <material name="realsense_body">
+        <color rgba="0.15 0.15 0.15 1.0"/>
       </material>
     </visual>
     <inertial>
-      <mass value="0.05"/>
-      <inertia ixx="0.000001" iyy="0.000001" izz="0.000001"
+      <mass value="0.072"/>  <!-- D435 mass: 72 g -->
+      <inertia ixx="0.000038" iyy="0.000005" izz="0.000038"
                ixy="0" ixz="0" iyz="0"/>
     </inertial>
   </link>
   <joint name="camera_joint" type="fixed">
-    <parent link="Gripper_1"/>
+    <parent link="base_link"/>
     <child link="camera_link"/>
-    <!-- 6 cm forward along gripper X, 4 cm above, pitched 30° down toward grasp -->
-    <origin xyz="0.06 0.0 0.04" rpy="0 0.5236 0"/>
+    <!-- Mounted behind and above the base, pitched forward to cover workspace.
+         Tune xyz/rpy here if you physically relocate the camera. -->
+    <origin xyz="-0.08 0.0 0.18" rpy="0 0.35 0"/>
   </joint>
-  <!-- ROS optical frame: Z forward, X right, Y down -->
+  <!-- ROS optical frame convention: Z forward, X right, Y down.
+       The -90° rotation around Z then -90° around X transforms from
+       the URDF body frame (X forward) to the ROS optical convention. -->
   <link name="camera_optical_frame"/>
   <joint name="camera_optical_joint" type="fixed">
@@ -173,24 +189,31 @@
     <origin xyz="0 0 0" rpy="-1.5708 0 -1.5708"/>
   </joint>
-  <!-- RGBD sensor (Gazebo Harmonic).                                      -->
-  <!-- Near clip 0.05 m suits close-range grasping; far 1.5 m covers the  -->
-  <!-- full reachable workspace of the Arctos arm.                         -->
+  <!-- Intel RealSense D435 RGBD sensor (Gazebo Harmonic).
+       Parameters match the D435 848×480 depth streaming mode.
+       The rgbd_camera sensor publishes colour image, depth image,
+       camera_info and a dense PointCloud2 under the <topic> prefix. -->
   <gazebo reference="camera_optical_frame">
-    <sensor name="depth_camera" type="rgbd_camera">
+    <sensor name="d435" type="rgbd_camera">
       <camera>
-        <horizontal_fov>1.047</horizontal_fov>  <!-- 60° FOV -->
+        <!-- D435 depth sensor horizontal FOV at 848×480: 86° -->
+        <horizontal_fov>1.5009</horizontal_fov>
         <image>
-          <width>640</width>
+          <!-- 848×480 — standard D435 streaming resolution -->
+          <width>848</width>
           <height>480</height>
           <format>R8G8B8</format>
         </image>
         <clip>
-          <near>0.05</near>
-          <far>1.5</far>
+          <!-- D435 minimum reliable depth: 0.105 m -->
+          <near>0.105</near>
+          <!-- Practical indoor range; D435 spec is up to ~10 m -->
+          <far>10.0</far>
         </clip>
         <noise>
+          <!-- Depth noise: D435 accuracy is ~2 % at 1 m → ~0.02 m.
+               σ = 0.003 m gives a realistic baseline for close-range work. -->
           <type>gaussian</type>
           <mean>0.0</mean>
-          <stddev>0.007</stddev>
+          <stddev>0.003</stddev>
         </noise>
       </camera>
