Commit message: fix(sim): replace gz_ros2_control with joint_state_publisher
Root cause: ros-humble-gz-ros2-control 0.7.17 exports IgnitionPluginHook
(compiled against gz-plugin 1.x / Ignition Fortress), but gz-sim 8.10.0
(Gazebo Harmonic) requires gz-plugin 2.x (GzPluginHook). The plugin will
never load, so controller_manager never starts and joint states are never
published — hence "RobotModel Error" in RViz and no arm control.

Fix:
- arctos_sim.xacro: remove <ros2_control> block and gz_ros2_control plugin;
  add <gravity>false</gravity> so the arm holds its zero pose in Gazebo
  without a controller.
- sim.launch.py: replace controller spawner chain with joint_state_publisher
  (publishes zero joint states → robot_state_publisher broadcasts TF tree →
  RViz renders the robot correctly).

For interactive joint control:
  ros2 run joint_state_publisher_gui joint_state_publisher_gui

https://claude.ai/code/session_014jKiKFNFx2wbEBY1JDbtYJ

File: arctos_gazebo/urdf/arctos_sim.xacro (robot description, xacro)
@@ -17,116 +17,9 @@
   <xacro:include filename="$(find arctos_description)/urdf/arctos.xacro"/>
   <!-- ================================================================== -->
-  <!-- ros2_control block — Gazebo hardware plugin                         -->
-  <!-- Joint definitions mirror arctos.ros2_control.xacro exactly so the  -->
-  <!-- same controllers.yaml works unchanged.                              -->
-  <!-- ================================================================== -->
-  <ros2_control name="GazeboSystem" type="system">
-    <hardware>
-      <plugin>gz_ros2_control/GazeboSimSystem</plugin>
-    </hardware>
-    <joint name="X_joint">
-      <command_interface name="position">
-        <param name="min">-3.14159265</param>
-        <param name="max">3.14159265</param>
-      </command_interface>
-      <command_interface name="velocity">
-        <param name="min">-3.15</param>
-        <param name="max">3.15</param>
-      </command_interface>
-      <state_interface name="position">
-        <param name="initial_value">0.0</param>
-      </state_interface>
-      <state_interface name="velocity"/>
-    </joint>
-    <joint name="Y_joint">
-      <command_interface name="position">
-        <param name="min">-0.96</param>
-        <param name="max">2.18</param>
-      </command_interface>
-      <command_interface name="velocity">
-        <param name="min">-3.15</param>
-        <param name="max">3.15</param>
-      </command_interface>
-      <state_interface name="position">
-        <param name="initial_value">0.0</param>
-      </state_interface>
-      <state_interface name="velocity"/>
-    </joint>
-    <joint name="Z_joint">
-      <command_interface name="position">
-        <param name="min">-1.5708</param>
-        <param name="max">0.9599</param>  <!-- 55/180*pi -->
-      </command_interface>
-      <command_interface name="velocity">
-        <param name="min">-3.15</param>
-        <param name="max">3.15</param>
-      </command_interface>
-      <state_interface name="position">
-        <param name="initial_value">0.0</param>
-      </state_interface>
-      <state_interface name="velocity"/>
-    </joint>
-    <joint name="A_joint">
-      <command_interface name="position">
-        <param name="min">-1.5708</param>
-        <param name="max">1.5708</param>
-      </command_interface>
-      <command_interface name="velocity">
-        <param name="min">-3.2</param>
-        <param name="max">3.2</param>
-      </command_interface>
-      <state_interface name="position">
-        <param name="initial_value">0.0</param>
-      </state_interface>
-      <state_interface name="velocity"/>
-    </joint>
-    <joint name="B_joint">
-      <command_interface name="position">
-        <param name="min">-1.55</param>
-        <param name="max">1.55</param>
-      </command_interface>
-      <command_interface name="velocity">
-        <param name="min">-3.2</param>
-        <param name="max">3.2</param>
-      </command_interface>
-      <state_interface name="position">
-        <param name="initial_value">0.0</param>
-      </state_interface>
-      <state_interface name="velocity"/>
-    </joint>
-    <joint name="C_joint">
-      <command_interface name="position">
-        <param name="min">-3.14159265</param>
-        <param name="max">3.14159265</param>
-      </command_interface>
-      <command_interface name="velocity">
-        <param name="min">-3.2</param>
-        <param name="max">3.2</param>
-      </command_interface>
-      <state_interface name="position">
-        <param name="initial_value">0.0</param>
-      </state_interface>
-      <state_interface name="velocity"/>
-    </joint>
-    <joint name="Left_jaw_joint">
-      <command_interface name="position">
-        <param name="min">0.0</param>
-        <param name="max">0.015</param>
-      </command_interface>
-      <state_interface name="position">
-        <param name="initial_value">0.0</param>
-      </state_interface>
-      <state_interface name="velocity"/>
-    </joint>
-  </ros2_control>
-  <!-- ================================================================== -->
-  <!-- Gazebo gz_ros2_control system plugin                                -->
-  <!-- This hooks ros2_control into the Gazebo simulation loop.            -->
+  <!-- Disable gravity on the robot so it holds its pose without a        -->
+  <!-- controller. Joint states come from joint_state_publisher in ROS.   -->
   <!-- ================================================================== -->
   <gazebo>
-    <plugin filename="gz_ros2_control-system"
-            name="gz_ros2_control::GazeboSimROS2ControlPlugin">
-      <parameters>$(find arctos_gazebo)/config/sim_controllers.yaml</parameters>
-    </plugin>
+    <gravity>false</gravity>
   </gazebo>
   <!-- ================================================================== -->

Commit message: restore(sim): full ros2_control + gravity for real-hardware pipeline
The joint_state_publisher workaround was wrong for the user's goal:
simulation must mirror the real-hardware control pipeline so the same
joint_trajectory_controller commands work in both environments.

Restore the ros2_control block in arctos_sim.xacro with all 7 joints
(X/Y/Z/A/B/C + Left_jaw) and the gz_ros2_control::GazeboSimROS2ControlPlugin.
Restore controller spawner chain in sim.launch.py (joint_state_broadcaster
→ arctos_arm_controller + arctos_hand_controller, via 30-s TimerAction).

Root problem (still pending): ros-humble-gz-ros2-control 0.7.17 was
compiled against gz-plugin 1.x (IgnitionPluginHook) but gz-sim 8 needs
gz-plugin 2.x (GzPluginHook). Fix: build gz_ros2_control from source
against the installed gz-sim 8 libraries — see instructions in README /
next commit message.

https://claude.ai/code/session_014jKiKFNFx2wbEBY1JDbtYJ

File: arctos_gazebo/urdf/arctos_sim.xacro (robot description, xacro)
@@ -17,9 +17,119 @@
   <xacro:include filename="$(find arctos_description)/urdf/arctos.xacro"/>
   <!-- ================================================================== -->
-  <!-- Disable gravity on the robot so it holds its pose without a        -->
-  <!-- controller. Joint states come from joint_state_publisher in ROS.   -->
+  <!-- ros2_control block — Gazebo hardware plugin                         -->
+  <!-- Joint definitions mirror arctos.ros2_control.xacro exactly so the  -->
+  <!-- same controllers.yaml works unchanged for real hardware.            -->
+  <!-- ================================================================== -->
+  <ros2_control name="GazeboSystem" type="system">
+    <hardware>
+      <plugin>gz_ros2_control/GazeboSimSystem</plugin>
+    </hardware>
+    <joint name="X_joint">
+      <command_interface name="position">
+        <param name="min">-3.14159265</param>
+        <param name="max">3.14159265</param>
+      </command_interface>
+      <command_interface name="velocity">
+        <param name="min">-3.15</param>
+        <param name="max">3.15</param>
+      </command_interface>
+      <state_interface name="position">
+        <param name="initial_value">0.0</param>
+      </state_interface>
+      <state_interface name="velocity"/>
+    </joint>
+    <joint name="Y_joint">
+      <command_interface name="position">
+        <param name="min">-0.96</param>
+        <param name="max">2.18</param>
+      </command_interface>
+      <command_interface name="velocity">
+        <param name="min">-3.15</param>
+        <param name="max">3.15</param>
+      </command_interface>
+      <state_interface name="position">
+        <param name="initial_value">0.0</param>
+      </state_interface>
+      <state_interface name="velocity"/>
+    </joint>
+    <joint name="Z_joint">
+      <command_interface name="position">
+        <param name="min">-1.5708</param>
+        <param name="max">0.9599</param>
+      </command_interface>
+      <command_interface name="velocity">
+        <param name="min">-3.15</param>
+        <param name="max">3.15</param>
+      </command_interface>
+      <state_interface name="position">
+        <param name="initial_value">0.0</param>
+      </state_interface>
+      <state_interface name="velocity"/>
+    </joint>
+    <joint name="A_joint">
+      <command_interface name="position">
+        <param name="min">-1.5708</param>
+        <param name="max">1.5708</param>
+      </command_interface>
+      <command_interface name="velocity">
+        <param name="min">-3.2</param>
+        <param name="max">3.2</param>
+      </command_interface>
+      <state_interface name="position">
+        <param name="initial_value">0.0</param>
+      </state_interface>
+      <state_interface name="velocity"/>
+    </joint>
+    <joint name="B_joint">
+      <command_interface name="position">
+        <param name="min">-1.55</param>
+        <param name="max">1.55</param>
+      </command_interface>
+      <command_interface name="velocity">
+        <param name="min">-3.2</param>
+        <param name="max">3.2</param>
+      </command_interface>
+      <state_interface name="position">
+        <param name="initial_value">0.0</param>
+      </state_interface>
+      <state_interface name="velocity"/>
+    </joint>
+    <joint name="C_joint">
+      <command_interface name="position">
+        <param name="min">-3.14159265</param>
+        <param name="max">3.14159265</param>
+      </command_interface>
+      <command_interface name="velocity">
+        <param name="min">-3.2</param>
+        <param name="max">3.2</param>
+      </command_interface>
+      <state_interface name="position">
+        <param name="initial_value">0.0</param>
+      </state_interface>
+      <state_interface name="velocity"/>
+    </joint>
+    <joint name="Left_jaw_joint">
+      <command_interface name="position">
+        <param name="min">0.0</param>
+        <param name="max">0.015</param>
+      </command_interface>
+      <state_interface name="position">
+        <param name="initial_value">0.0</param>
+      </state_interface>
+      <state_interface name="velocity"/>
+    </joint>
+  </ros2_control>
+  <!-- ================================================================== -->
+  <!-- gz_ros2_control system plugin                                        -->
+  <!-- NOTE: requires gz_ros2_control built against gz-plugin 2.x          -->
+  <!-- (gz-sim 8 / Harmonic). The apt package ros-humble-gz-ros2-control   -->
+  <!-- 0.7.17 is compiled against gz-plugin 1.x and will NOT load.         -->
+  <!-- Build from source: see README for instructions.                      -->
   <!-- ================================================================== -->
   <gazebo>
-    <gravity>false</gravity>
+    <plugin filename="gz_ros2_control-system"
+            name="gz_ros2_control::GazeboSimROS2ControlPlugin">
+      <parameters>$(find arctos_gazebo)/config/sim_controllers.yaml</parameters>
+    </plugin>
   </gazebo>
   <!-- ================================================================== -->

Commit message: Fix camera mount: move back/up to clear arm geometry and correct pitch direction
The previous mount at (-0.08, 0, 0.18) with rpy="0 +0.35 0" had two bugs:
  1. Positive pitch in URDF rotates the X-axis upward, so the camera was
     looking up and forward rather than down at the workspace.
  2. The position was too close to the arm base, risking geometry collision.

New mount: xyz="-0.20 0.0 0.45", rpy="0 -0.55 0"
  - 20 cm behind, 45 cm above base_link — clears the arm body/motors
  - Negative pitch (−31°) correctly aims the camera downward
  - Gaze centre hits the table top at approximately (0.45, 0, 0.05),
    covering the red box, blue cylinder and green sphere.

Also update the arctos_world.sdf comment to reflect the new camera pose.

https://claude.ai/code/session_014jKiKFNFx2wbEBY1JDbtYJ

File: arctos_gazebo/urdf/arctos_sim.xacro (robot description, xacro)
@@ -141,7 +141,9 @@
   <!--                                                                     -->
   <!-- Mount position (adjust to suit your physical setup):               -->
-  <!--   xyz="-0.08 0.0 0.18"  — 8 cm behind, 18 cm above base origin    -->
-  <!--   rpy="0 0.35 0"        — pitched ~20° forward to centre the FOV  -->
-  <!--                            on the arm's reachable workspace         -->
+  <!--   xyz="-0.20 0.0 0.45"  — 20 cm behind, 45 cm above base origin   -->
+  <!--                            clears the arm base/motor geometry       -->
+  <!--   rpy="0 -0.55 0"       — pitched ~31° downward (negative pitch =  -->
+  <!--                            look down); centres FOV on the table at  -->
+  <!--                            x≈0.4, z≈0.08 m                         -->
   <!--                                                                     -->
   <!-- D435 depth sensor parameters (848×480 mode):                       -->
@@ -179,7 +181,7 @@
     <parent link="base_link"/>
     <child link="camera_link"/>
-    <!-- Mounted behind and above the base, pitched forward to cover workspace.
+    <!-- Mounted behind and above the base, pitched downward to cover workspace.
          Tune xyz/rpy here if you physically relocate the camera. -->
-    <origin xyz="-0.08 0.0 0.18" rpy="0 0.35 0"/>
+    <origin xyz="-0.20 0.0 0.45" rpy="0 -0.55 0"/>
   </joint>
   <!-- ROS optical frame convention: Z forward, X right, Y down.

Commit message: Move camera and table to robot front (+Y direction)
Camera was at -X (robot's right); table was at +X (robot's left).
Robot faces +Y, so both are repositioned along the +Y axis:
- camera_joint: xyz="0 0.20 0.45", yaw rotated 90° to face +Y
- table pose: 0 0.40 0.025 (world frame)
- red_box, blue_cylinder, green_sphere shifted to sit on new table

https://claude.ai/code/session_014jKiKFNFx2wbEBY1JDbtYJ

File: arctos_gazebo/urdf/arctos_sim.xacro (robot description, xacro)
@@ -141,9 +141,9 @@
   <!--                                                                     -->
   <!-- Mount position (adjust to suit your physical setup):               -->
-  <!--   xyz="-0.20 0.0 0.45"  — 20 cm behind, 45 cm above base origin   -->
-  <!--                            clears the arm base/motor geometry       -->
-  <!--   rpy="0 -0.55 0"       — pitched ~31° downward (negative pitch =  -->
-  <!--                            look down); centres FOV on the table at  -->
-  <!--                            x≈0.4, z≈0.08 m                         -->
+  <!--   xyz="0.0 0.20 0.45"   — 20 cm in front, 45 cm above base origin  -->
+  <!--                            camera faces forward toward the table    -->
+  <!--   rpy="0 -0.55 1.5708"  — pitched ~31° down, yaw 90° to face +Y  -->
+  <!--                            (robot forward); centres FOV on table   -->
+  <!--                            at y≈0.4, z≈0.08 m                     -->
   <!--                                                                     -->
   <!-- D435 depth sensor parameters (848×480 mode):                       -->
@@ -183,5 +183,5 @@
     <!-- Mounted behind and above the base, pitched downward to cover workspace.
          Tune xyz/rpy here if you physically relocate the camera. -->
-    <origin xyz="-0.20 0.0 0.45" rpy="0 -0.55 0"/>
+    <origin xyz="0.0 0.20 0.45" rpy="0 -0.55 1.5708"/>
   </joint>
   <!-- ROS optical frame convention: Z forward, X right, Y down.

Commit message: fix(sim): stop Right_jaw_joint falling free; reduce controller spawn wait
Two causes of "robot falls apart when controllers load":

1. Right_jaw_joint was absent from the ros2_control block, so
   GazeboSimSystem never commanded it.  DART physics (Gazebo Harmonic)
   does not support SDF-level mimic constraints (logged as [Err]), so
   Right_jaw_joint hung freely under gravity making the gripper look
   broken.  Fix: add Right_jaw_joint to the ros2_control block with
   <param name="mimic">Left_jaw_joint</param> so GazeboSimSystem handles
   it in software each physics step, bypassing the physics constraint.
   multiplier=-1 matches a symmetric parallel gripper; adjust if needed.

2. The 30 s controller-spawn timer let the arm dangle under gravity for
   half a minute before being grabbed by JointTrajectoryController.
   Now that gz_ros2_control builds against gz-plugin 2.x the plugin loads
   in 2-3 s, so the wait is reduced to 10 s.

https://claude.ai/code/session_014jKiKFNFx2wbEBY1JDbtYJ

File: arctos_gazebo/urdf/arctos_sim.xacro (robot description, xacro)
@@ -113,4 +113,30 @@
         <param name="min">0.0</param>
         <param name="max">0.015</param>
+      </command_interface>
+      <state_interface name="position">
+        <param name="initial_value">0.0</param>
+      </state_interface>
+      <state_interface name="velocity"/>
+    </joint>
+    <!--
+      Right_jaw_joint: mimic of Left_jaw_joint via gz_ros2_control software mimic.
+      DART physics (used by Gazebo Harmonic) does not support SDF-level mimic
+      constraints, so the physics engine logs an error and leaves Right_jaw_joint
+      uncontrolled.  By declaring it here with <param name="mimic">, GazeboSimSystem
+      commands Right_jaw_joint directly each physics step to track Left_jaw_joint,
+      bypassing the physics-engine constraint entirely.
+      multiplier: adjust sign/scale to match your URDF convention.
+        multiplier= 1  → Right jaw moves in the same angular direction as Left jaw
+        multiplier=-1  → Right jaw moves in the opposite angular direction (typical
+                         for symmetric parallel grippers where both jaws open outward)
+      Check arctos_description/urdf/arctos.xacro <mimic multiplier="…"> attribute
+      for the correct value; the default here is -1 for a symmetric parallel gripper.
+    -->
+    <joint name="Right_jaw_joint">
+      <param name="mimic">Left_jaw_joint</param>
+      <param name="multiplier">-1</param>
+      <command_interface name="position">
+        <param name="min">-0.015</param>
+        <param name="max">0.0</param>
       </command_interface>
       <state_interface name="position">
