Commit message: fix(sim): switch arm joints to effort interface + JTC PID gains
Previous attempts used position command interface, which gz_ros2_control
Harmonic implements via JointPositionReset — a per-step kinematic teleport.
JointPositionReset is unreliable when DART has accumulated joint velocity:
the teleport fights the existing velocity and creates a large constraint
impulse that violates joint constraints and causes links to fly apart.
The <param name="p/d"> values added previously are a Gazebo Classic
(gazebo_ros2_control) artifact and are silently ignored in gz_ros2_control.

Fix — effort command interface throughout the arm:
  arctos_sim.xacro: all six arm joints now expose only
    <command_interface name="effort"/>
  The gripper joints (Left_jaw_joint, Right_jaw_joint) keep position.

  sim_controllers.yaml: arctos_arm_controller now uses
    command_interfaces: [effort]
  with an explicit gains: block per joint:
    Y_joint (shoulder): p=1000 d=100  — highest gravity load
    Z_joint (elbow):    p=600  d=60
    X_joint (base):     p=500  d=50
    A_joint, B_joint:   p=200  d=20   — wrist
    C_joint:            p=100  d=10   — tool roll
    i=0 on all joints (integral windup destabilises DART).

  open_loop_control removed: with effort interface we want full position
  feedback so the PID error signal counteracts gravity.

Control path is now:
  JTC → effort = Kp*(q_des-q) + Kd*(dq_des-dq) → GazeboSimSystem
  → JointForceCmd → DART integrator (torque injected, not teleported)

https://claude.ai/code/session_014jKiKFNFx2wbEBY1JDbtYJ

File: arctos_gazebo/urdf/arctos_sim.xacro (robot description, xacro)
@@ -26,124 +26,48 @@
     </hardware>
     <!--
-      PD gains for GazeboSimSystem position control.
-      GazeboSimSystem converts position commands to joint forces via a PD
-      loop: force = p*(q_cmd - q) + d*(dq_cmd - dq).  Without these params
-      both gains default to 0 and the controller applies zero force — the
-      arm falls under gravity regardless of what the trajectory controller
-      commands.
-      Tuning guide (scale proportionally to link mass × reach²):
-        p  — stiffness.  Too low → arm droops under gravity.
-             Too high → high-frequency oscillation.
-        d  — damping.  ~10 % of p is a safe starting point.
-             Too low → ringing.  Too high → sluggish / overdamped.
-        i  — leave at 0 for simulation; integral windup destabilises DART.
-      These gains are SIMULATION-ONLY and have no effect on real hardware.
+      Arm joints use EFFORT command interface.
+      GazeboSimSystem passes the effort command directly to DART as a joint
+      torque via JointForceCmd — no internal PID, no kinematic tricks.
+      The PID loop (position error → effort) lives in the JointTrajectoryController
+      and is configured in sim_controllers.yaml under gains:.
+      Why NOT position interface?
+        In gz_ros2_control for gz-sim Harmonic, position commands are applied
+        via JointPositionReset, a kinematic teleport.  If DART has accumulated
+        even a small joint velocity beforehand, the teleport creates a large
+        constraint impulse that can violate joint constraints and cause links
+        to fly apart.  Additionally, the <param name="p/d"> values in the URDF
+        <joint> block are a Gazebo Classic artifact — gz_ros2_control ignores them.
+      With effort interface, the torque is injected into DART's integrator
+      each step.  Gravity is counteracted by the PID error signal.  No
+      teleportation, no constraint impulse, no flying links.
     -->
-    <!-- X_joint — base yaw: moderate load (whole-arm inertia about vertical) -->
     <joint name="X_joint">
-      <param name="p">500</param>
-      <param name="i">0</param>
-      <param name="d">50</param>
-      <command_interface name="position">
-        <param name="min">-3.14159265</param>
-        <param name="max">3.14159265</param>
-      </command_interface>
-      <command_interface name="velocity">
-        <param name="min">-3.15</param>
-        <param name="max">3.15</param>
-      </command_interface>
-      <state_interface name="position">
-        <param name="initial_value">0.0</param>
-      </state_interface>
-      <state_interface name="velocity"/>
-    </joint>
-    <!-- Y_joint — shoulder pitch: highest gravity torque, needs stiffest gains -->
+      <command_interface name="effort"/>
+      <state_interface name="position"><param name="initial_value">0.0</param></state_interface>
+      <state_interface name="velocity"/>
+    </joint>
     <joint name="Y_joint">
-      <param name="p">1000</param>
-      <param name="i">0</param>
-      <param name="d">100</param>
-      <command_interface name="position">
-        <param name="min">-0.96</param>
-        <param name="max">2.18</param>
-      </command_interface>
-      <command_interface name="velocity">
-        <param name="min">-3.15</param>
-        <param name="max">3.15</param>
-      </command_interface>
-      <state_interface name="position">
-        <param name="initial_value">0.0</param>
-      </state_interface>
-      <state_interface name="velocity"/>
-    </joint>
-    <!-- Z_joint — elbow pitch: significant gravity torque from forearm + wrist -->
+      <command_interface name="effort"/>
+      <state_interface name="position"><param name="initial_value">0.0</param></state_interface>
+      <state_interface name="velocity"/>
+    </joint>
     <joint name="Z_joint">
-      <param name="p">600</param>
-      <param name="i">0</param>
-      <param name="d">60</param>
-      <command_interface name="position">
-        <param name="min">-1.5708</param>
-        <param name="max">0.9599</param>
-      </command_interface>
-      <command_interface name="velocity">
-        <param name="min">-3.15</param>
-        <param name="max">3.15</param>
-      </command_interface>
-      <state_interface name="position">
-        <param name="initial_value">0.0</param>
-      </state_interface>
-      <state_interface name="velocity"/>
-    </joint>
-    <!-- A_joint — wrist pitch: light load (wrist + gripper only) -->
+      <command_interface name="effort"/>
+      <state_interface name="position"><param name="initial_value">0.0</param></state_interface>
+      <state_interface name="velocity"/>
+    </joint>
     <joint name="A_joint">
-      <param name="p">200</param>
-      <param name="i">0</param>
-      <param name="d">20</param>
-      <command_interface name="position">
-        <param name="min">-1.5708</param>
-        <param name="max">1.5708</param>
-      </command_interface>
-      <command_interface name="velocity">
-        <param name="min">-3.2</param>
-        <param name="max">3.2</param>
-      </command_interface>
-      <state_interface name="position">
-        <param name="initial_value">0.0</param>
-      </state_interface>
-      <state_interface name="velocity"/>
-    </joint>
-    <!-- B_joint — wrist roll: negligible gravity torque, moderate damping -->
+      <command_interface name="effort"/>
+      <state_interface name="position"><param name="initial_value">0.0</param></state_interface>
+      <state_interface name="velocity"/>
+    </joint>
     <joint name="B_joint">
-      <param name="p">200</param>
-      <param name="i">0</param>
-      <param name="d">20</param>
-      <command_interface name="position">
-        <param name="min">-1.55</param>
-        <param name="max">1.55</param>
-      </command_interface>
-      <command_interface name="velocity">
-        <param name="min">-3.2</param>
-        <param name="max">3.2</param>
-      </command_interface>
-      <state_interface name="position">
-        <param name="initial_value">0.0</param>
-      </state_interface>
-      <state_interface name="velocity"/>
-    </joint>
-    <!-- C_joint — tool roll: end-of-chain, very light load -->
+      <command_interface name="effort"/>
+      <state_interface name="position"><param name="initial_value">0.0</param></state_interface>
+      <state_interface name="velocity"/>
+    </joint>
     <joint name="C_joint">
-      <param name="p">100</param>
-      <param name="i">0</param>
-      <param name="d">10</param>
-      <command_interface name="position">
-        <param name="min">-3.14159265</param>
-        <param name="max">3.14159265</param>
-      </command_interface>
-      <command_interface name="velocity">
-        <param name="min">-3.2</param>
-        <param name="max">3.2</param>
-      </command_interface>
-      <state_interface name="position">
-        <param name="initial_value">0.0</param>
-      </state_interface>
+      <command_interface name="effort"/>
+      <state_interface name="position"><param name="initial_value">0.0</param></state_interface>
       <state_interface name="velocity"/>
     </joint>

Commit message: fix(sim): switch to position interface — root cause of joint falling apart
Root cause analysis
───────────────────
The reference URDF (arctos.xacro) already defines:

    <link name="world" />
    <joint name="world_joint" type="fixed">
        <parent link="world"/>
        <child link="base_link"/>
    </joint>

robot_state_publisher therefore publishes world→base_link automatically
from the fixed joint — the separate static_transform_publisher was a
duplicate that caused TF conflicts.

The deeper cause of the joint flying apart was the effort command
interface.  With effort interface, JointTrajectoryController must
counteract gravity entirely through PID error torques.  Between startup
and the first controller update cycle, DART integrates one step under
gravity with zero effort command — enough to impart velocity and trigger
a DART impulse response on the next step, which can violate a joint
constraint and make a link visually separate.

The real ArctosInterface (hardware) used POSITION command interface.
In gz_ros2_control, position commands are applied via JointPositionReset:
DART's joint q is overwritten kinematically each step.  There is no
integration under gravity, no impulse, no drooping.  The arm holds 0 rad
from the very first PreUpdate call regardless of when physics starts.

Changes
───────
arctos_sim.xacro
  • All 6 arm joints: effort → position command interface (with limits)
  • Updated comment to explain why position interface is correct

sim_controllers.yaml
  • command_interfaces: [effort] → [position]
  • Removed entire gains: section (not needed for position interface)

sim.launch.py
  • Gazebo now started with -r (auto-run); no delayed-unpause needed
  • Removed static_transform_publisher (RSP handles world→base_link via
    world_joint in the URDF)
  • Removed homing_cmd, unpause_world, on_arm_active, home_arg, TimerAction
  • Spawn pose reverted to 0 0 0 (z=0.001 offset was a bandaid for effort)
  • Launch file is now ~170 lines shorter and has no timing dependencies

https://claude.ai/code/session_014jKiKFNFx2wbEBY1JDbtYJ

File: arctos_gazebo/urdf/arctos_sim.xacro (robot description, xacro)
@@ -18,6 +18,6 @@
   <!-- ================================================================== -->
   <!-- ros2_control block — Gazebo hardware plugin                         -->
-  <!-- Joint definitions mirror arctos.ros2_control.xacro exactly so the  -->
-  <!-- same controllers.yaml works unchanged for real hardware.            -->
+  <!-- Mirrors arctos.ros2_control.xacro (real hardware) interface types  -->
+  <!-- so the same controllers.yaml structure works in both contexts.      -->
   <!-- ================================================================== -->
   <ros2_control name="GazeboSystem" type="system">
@@ -26,47 +26,62 @@
     </hardware>
     <!--
-      Arm joints use EFFORT command interface.
-      GazeboSimSystem passes the effort command directly to DART as a joint
-      torque via JointForceCmd — no internal PID, no kinematic tricks.
-      The PID loop (position error → effort) lives in the JointTrajectoryController
-      and is configured in sim_controllers.yaml under gains:.
-      Why NOT position interface?
-        In gz_ros2_control for gz-sim Harmonic, position commands are applied
-        via JointPositionReset, a kinematic teleport.  If DART has accumulated
-        even a small joint velocity beforehand, the teleport creates a large
-        constraint impulse that can violate joint constraints and cause links
-        to fly apart.  Additionally, the <param name="p/d"> values in the URDF
-        <joint> block are a Gazebo Classic artifact — gz_ros2_control ignores them.
-      With effort interface, the torque is injected into DART's integrator
-      each step.  Gravity is counteracted by the PID error signal.  No
-      teleportation, no constraint impulse, no flying links.
+      Arm joints use POSITION command interface — same as real hardware.
+      GazeboSimSystem applies position commands via JointPositionReset in
+      DART, which kinematically sets the joint position each physics step.
+      This matches what the real ArctosInterface does (motor servo to a
+      target position).  It is unconditionally stable at startup: the JTC
+      sends q_des=0 from the very first PreUpdate call, so DART never has a
+      chance to let gravity move the joints.  No PID tuning, no gravity
+      compensation, no timing gymnastics required.
+      arctos.xacro already contains "world_joint" (fixed, world→base_link)
+      so DART treats the base as rigidly anchored — not free-floating.
+      robot_state_publisher publishes the world→base_link TF automatically
+      from this fixed joint; no separate static_transform_publisher needed.
     -->
     <joint name="X_joint">
-      <command_interface name="effort"/>
+      <command_interface name="position">
+        <param name="min">-3.14159</param>
+        <param name="max"> 3.14159</param>
+      </command_interface>
       <state_interface name="position"><param name="initial_value">0.0</param></state_interface>
       <state_interface name="velocity"/>
     </joint>
     <joint name="Y_joint">
-      <command_interface name="effort"/>
+      <command_interface name="position">
+        <param name="min">-0.96</param>
+        <param name="max"> 2.18</param>
+      </command_interface>
       <state_interface name="position"><param name="initial_value">0.0</param></state_interface>
       <state_interface name="velocity"/>
     </joint>
     <joint name="Z_joint">
-      <command_interface name="effort"/>
+      <command_interface name="position">
+        <param name="min">-1.5708</param>
+        <param name="max"> 0.9599</param>
+      </command_interface>
       <state_interface name="position"><param name="initial_value">0.0</param></state_interface>
       <state_interface name="velocity"/>
     </joint>
     <joint name="A_joint">
-      <command_interface name="effort"/>
+      <command_interface name="position">
+        <param name="min">-1.5708</param>
+        <param name="max"> 1.5708</param>
+      </command_interface>
       <state_interface name="position"><param name="initial_value">0.0</param></state_interface>
       <state_interface name="velocity"/>
     </joint>
     <joint name="B_joint">
-      <command_interface name="effort"/>
+      <command_interface name="position">
+        <param name="min">-1.55</param>
+        <param name="max"> 1.55</param>
+      </command_interface>
       <state_interface name="position"><param name="initial_value">0.0</param></state_interface>
       <state_interface name="velocity"/>
     </joint>
     <joint name="C_joint">
-      <command_interface name="effort"/>
+      <command_interface name="position">
+        <param name="min">-3.14159</param>
+        <param name="max"> 3.14159</param>
+      </command_interface>
       <state_interface name="position"><param name="initial_value">0.0</param></state_interface>
       <state_interface name="velocity"/>
